File: pcb/revB/karabas-opl3.kicad_pcb (KiCad board)
At the start: 2 copper layers, 92.2 x 44 mm, 73 parts, among them J1 Conn_02x05_Odd_Even, J2 Conn_02x30_Row_Letter_First, J3 PJ307, J4 Conn_01x04, J5 5V_PRG, U1 YMF262-M, U2 74AHCT1G125DB, U3 EPM3128ATC100, U4 UDA1334ATS, U5 1117-3.3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

Commit message: Updated revB gerbers
Routing:
- net +5V: track 150.7 -> 150.6 mm, vias 14 -> 16
- net GNDA: vias 11 -> 13
- net GND: vias 54 -> 63
